Commit message: Added resource vehicle: listen to its tf

File: models/rexrov/urdf/rexrov_base_resource.xacro (robot description, xacro)
@@ -88,5 +88,5 @@
         <origin xyz="0 0 0" rpy="0 0 0"/>
 	<geometry>
-          <box size="10 10 10"/>
+          <box size="6 6 2"/>
         </geometry>
       </visual>

Commit message: added 2nd resource, decrease resource size, add 2nd resource js1

File: models/rexrov/urdf/rexrov_base_resource.xacro (robot description, xacro)
@@ -88,5 +88,5 @@
         <origin xyz="0 0 0" rpy="0 0 0"/>
 	<geometry>
-          <box size="6 6 2"/>
+          <box size="1 1 1"/>
         </geometry>
       </visual>
